File: RFExperiments/Hardware/LT5560.sch (EAGLE design)
At the start: 47 parts, among them IC1 LT5560, IC2 LTC6362, IC3 VREG-TS1117CW-5V, Q1 BSS123, Q2 BSS123, X1 IN, X2 LO

Commit message: Bugfixes and tests
Parts:
- C12: value DNP -> 100n
Changed lines of the file:
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@@
 <part name="R8" library="rcl" deviceset="R-EU_" device="R0603" value="200"/>
 <part name="C11" library="resistor" deviceset="C-EU" device="C0603" value="DNP"/>
-<part name="C12" library="resistor" deviceset="C-EU" device="C0603" value="DNP"/>
+<part name="C12" library="resistor" deviceset="C-EU" device="C0603" value="100n"/>
 <part name="R9" library="rcl" deviceset="R-EU_" device="R0603" value="33"/>
 <part name="R10" library="rcl" deviceset="R-EU_" device="R0603" value="33"/>
