File: RFExperiments/Hardware/MAX2871.brd (EAGLE design)
At the start: 50 x 50 mm, 49 parts, among them IC1 AP2114H, IC2 MAX2871, IC4 NCP702-3.3, IC5 NCP702-3.3, X1 SMA_CONNECTOR, X2 SMA_CONNECTOR, X3 SMA_CONNECTOR, X4 SMA_CONNECTOR, X5 SMA_CONNECTOR

Commit message: Bugfixes and tests
Parts:
- C4: value 2n -> 180p
- C5: value 180p -> 18p
- C6: value 33n -> 3n3
- R1: value 1k -> 1k8
- R2: value 100 -> 82
- R3: value 120 -> 330
Changed lines of the file:
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@@
 <attribute name="VALUE" x="24.405" y="29.965" size="1.27" layer="27" rot="R90"/>
 </element>
-<element name="C4" library="rcl" package="C0603" value="2n" x="27.1" y="18" smashed="yes">
+<element name="C4" library="rcl" package="C0603" value="180p" x="27.1" y="18" smashed="yes">
 <attribute name="NAME" x="24.365" y="17.735" size="0.8128" layer="25" font="vector"/>
 <attribute name="VALUE" x="26.465" y="16.095" size="1.27" layer="27"/>
 </element>
-<element name="C5" library="rcl" package="C0603" value="180p" x="30" y="19.4" smashed="yes" rot="R270">
+<element name="C5" library="rcl" package="C0603" value="18p" x="30" y="19.4" smashed="yes" rot="R270">
 <attribute name="NAME" x="28.465" y="20.935" size="0.8128" layer="25" font="vector"/>
 <attribute name="VALUE" x="28.095" y="20.035" size="1.27" layer="27" rot="R270"/>
 </element>
-<element name="C6" library="rcl" package="C0603" value="33n" x="27.1" y="15.8" smashed="yes">
+<element name="C6" library="rcl" package="C0603" value="3n3" x="27.1" y="15.8" smashed="yes">
 <attribute name="NAME" x="24.365" y="15.435" size="0.8128" layer="25" font="vector"/>
 <attribute name="VALUE" x="26.465" y="13.895" size="1.27" layer="27"/>
@@
 <attribute name="VALUE" x="14.4" y="30.1" size="1.27" layer="27" rot="R90"/>
 </element>
-<element name="R1" library="resistor" package="R0603" value="1k" x="30" y="15.8" smashed="yes" rot="R90">
+<element name="R1" library="resistor" package="R0603" value="1k8" x="30" y="15.8" smashed="yes" rot="R90">
 <attribute name="NAME" x="29.965" y="12.965" size="0.8128" layer="25" font="vector" rot="R90"/>
 <attribute name="VALUE" x="31.905" y="15.165" size="1.27" layer="27" rot="R90"/>
@@
 <attribute name="VALUE" x="19.965" y="16.595" size="1.27" layer="27"/>
 </element>
-<element name="R2" library="resistor" package="R0603" value="100" x="27.1" y="13.6" smashed="yes" rot="R180">
+<element name="R2" library="resistor" package="R0603" value="82" x="27.1" y="13.6" smashed="yes" rot="R180">
 <attribute name="NAME" x="25.435" y="14.465" size="0.8128" layer="25" font="vector" rot="R180"/>
 <attribute name="VALUE" x="27.735" y="15.505" size="1.27" layer="27" rot="R180"/>
 </element>
-<element name="R3" library="resistor" package="R0603" value="120" x="27.1" y="11.4" smashed="yes">
+<element name="R3" library="resistor" package="R0603" value="330" x="27.1" y="11.4" smashed="yes">
 <attribute name="NAME" x="24.265" y="11.035" size="0.8128" layer="25" font="vector"/>
 <attribute name="VALUE" x="26.465" y="9.495" size="1.27" layer="27"/>
