File: RFExperiments/Hardware/MAX2871.sch (EAGLE design)
At the start: 49 parts, among them IC1 AP2114H, IC2 MAX2871, IC4 NCP702-3.3, IC5 NCP702-3.3, X1 SMA_CONNECTOR, X2 SMA_CONNECTOR, X3 SMA_CONNECTOR, X4 SMA_CONNECTOR, X5 SMA_CONNECTOR

Commit message: Bugfixes and tests
Parts:
- C4: value 2n -> 180p
- C5: value 180p -> 18p
- C6: value 33n -> 3n3
- R1: value 1k -> 1k8
- R2: value 100 -> 82
- R3: value 120 -> 330
Other:
- note added: "Approx. 450kHz loop bandwidth"
Changed lines of the file:
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@@
 <part name="IC2" library="rf" deviceset="MAX2871" device="" package3d_urn="urn:adsk.eagle:package:11260353/1"/>
 <part name="GND2" library="supply1" deviceset="GND" device=""/>
-<part name="R1" library="resistor" deviceset="R-EU_" device="R0603" value="1k"/>
-<part name="R2" library="resistor" deviceset="R-EU_" device="R0603" value="100"/>
-<part name="R3" library="resistor" deviceset="R-EU_" device="R0603" value="120"/>
+<part name="R1" library="resistor" deviceset="R-EU_" device="R0603" value="1k8"/>
+<part name="R2" library="resistor" deviceset="R-EU_" device="R0603" value="82"/>
+<part name="R3" library="resistor" deviceset="R-EU_" device="R0603" value="330"/>
 <part name="C1" library="rcl" deviceset="C-EU" device="C0603" value="1u"/>
 <part name="C2" library="rcl" deviceset="C-EU" device="C0603" value="1u"/>
 <part name="C3" library="rcl" deviceset="C-EU" device="C0603" value="1u"/>
-<part name="C4" library="rcl" deviceset="C-EU" device="C0603" value="2n"/>
-<part name="C5" library="rcl" deviceset="C-EU" device="C0603" value="180p"/>
-<part name="C6" library="rcl" deviceset="C-EU" device="C0603" value="33n"/>
+<part name="C4" library="rcl" deviceset="C-EU" device="C0603" value="180p"/>
+<part name="C5" library="rcl" deviceset="C-EU" device="C0603" value="18p"/>
+<part name="C6" library="rcl" deviceset="C-EU" device="C0603" value="3n3"/>
 <part name="GND3" library="supply1" deviceset="GND" device=""/>
 <part name="GND4" library="supply1" deviceset="GND" device=""/>
@@
 <text x="12.7" y="45.72" size="1.778" layer="97">All I/O using 3V3 levels</text>
 <text x="68.58" y="160.02" size="1.778" layer="97">3x 3V3</text>
+<text x="175.26" y="17.78" size="1.778" layer="97">Approx. 450kHz loop bandwidth</text>
 </plain>
 <instances>
