File: Hardware/VNA.brd (EAGLE design)
At the start: 160 x 100 mm, 316 parts, among them IC1 LTC5510, IC10 LT5560, IC11 LTC6362, IC12 MCP33131D-10-E/MS, IC13 SI5351C, IC14 MAX2871, IC15 NCP702-3.3, IC16 RFSW6042, IC17 AP2114H, IC18 RFSW6042, IC19 MAX2871, IC2 LT5560, IC20 NCP702-3.3, IC21 AP2114H, IC22 F2912, IC23 F1958, IC24 TRF37A73, IC25 F2912, IC26 F2912, IC27 F2912, IC3 LTC6362, IC4 MCP33131D-10-E/MS, IC5 LTC5510, IC6 LT5560, IC7 LTC6362, IC8 MCP33131D-10-E/MS, IC9 LTC5510, J1 U.FL-R-SMT, J2 U.FL-R-SMT, Q1 FA-128 26MHz, T1 MABA011082, T2 MABA011082, T3 MABA011082, X1 RLB DUT/RF IN, X2 RLB DUT/RF IN

Commit message: Placing
Parts:
- removed C106, C113: 100n, rcl:C0603
- moved L14 231.1 mm to (92.5, 34.0), turned to 90 degrees
- moved L13 221.7 mm to (87.5, 34.0), turned to 90 degrees
- moved R26 218.6 mm to (93.5, 21.7), flipped to the bottom
- moved C33 214.8 mm to (90.0, 6.00), turned to 90 degrees
- moved R28 214.7 mm to (89.2, 51.0)
- moved R29 213.2 mm to (84.5, 58.5), turned to 90 degrees
- moved R21 212.7 mm to (84.0, 5.00), turned to 270 degrees
- moved C34 209.2 mm to (78.0, 7.00)
- moved R27 208.7 mm to (88.5, 52.5)
- moved C87 208.7 mm to (77.5, 44.5), turned to 90 degrees
- moved R9 202.1 mm to (80.0, 9.00), turned to 270 degrees
- moved C64 199.2 mm to (86.0, 74.0)
- moved R25 196.0 mm to (95.0, 25.2)
- moved C63 191.9 mm to (85.0, 71.5), turned to 270 degrees
- moved C85 189.8 mm to (68.0, 64.5), turned to 90 degrees
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Connections:
- removed net N$100: C112.1, IC13.19, L37.1
- new net N$160: C112.1, IC13.17, L37.1
- net GND: no longer C106.1, C113.1
- net LO1_REF: now also IC13.9; no longer IC13.12
- net N$101: now also IC13.19; no longer IC13.9
- net N$109: no longer C106.2, C113.2
- net N$157: now also IC13.13; no longer IC13.17
- net N$23: now also T2.2; no longer T2.1
- net N$25: now also T2.1; no longer T2.2
- net N$97: now also IC13.12; no longer IC13.8
- net SOURCE_REF: now also IC13.8; no longer IC13.13
Other:
- board size 160 x 100 mm -> 100 x 100 mm

Commit message: Partial routing
Parts:
- removed R14, R26, R42: 51k, rcl:R0603
- added C106, C158, C160, C162, C164, C165, C166, C167, C168, C193, C194, C195: 1u, rcl:C0603
- added C113, C159, C161, C163: 4u7, rcl:C0603
- added C169, C170, C171, C172, C174, C180, C181, C184, C189, C190: 22u, rcl:C1206
- added C173, C177, C185: 10u/25V, rcl:C1206
- added C175, C178, C186: 47n, rcl:C0603
- added C176: 510p, rcl:C0603
- added C179, C183: DNP, rcl:C0603
- added C182: 120p, rcl:C0603
- added C187: 1n, rcl:C0603
- added C188: 8p2, rcl:C0603
- added C191, C192, C203, C204, C205, C206, C207, C208, C209, C210, C211: 100n, rcl:C0603
- added IC28, IC29, IC30, IC31: LDL212PU50R, custom-ic:SON95P300X300X100-7T170X240N
- added IC32: TPS65265, custom-ic:QFN50P500X500X100-33T345N
- added IC33: STM32L432KC, custom-ic:QFN50P500X500X100-33T345N
- added IC34, IC35, IC36: NCP702-1.8, rf:SOT95P240X110-5
- added J3: DCJ0202, con-jack:DCJ0202
- added JP1: (no value), pinhead:1X06
- added JTAG: (no value), con-ml:ML10
- added L47, L48, L49, L50: Ferrite, rf:R0603
- added L51, L55: 10u, custom-ic:SRN5040
- added L52, L53, L54: 6u8, custom-ic:SRN5040
- added R100, R101, R102, R103, R104, R90, R92, R93, R94, R95, R97, R98, R99: 10k, resistor:R0603
- added R76, R88, R91, R96: 22, resistor:R0603
- added R77: DNP, rcl:R0603
- added R78: 51k, rcl:R0603
- added R79: 82k, rcl:R0603
- added R80, R83, R86: 10k, rcl:R0603
- added R81: 91k, rcl:R0603
- added R82: 30k, rcl:R0603
- added R84: 45k3, rcl:R0603
- added R85: 16k, rcl:R0603
- added R87: 20k, rcl:R0603
- added R89: 1k5, resistor:R0603
- added U2: 6SLX9TQG144, xilinx_devices_V6:TQ144
- added U4: W25Q16BVSN, memory-winbond:SO08
- added X3: MINI-USB-32005-201, con-cypressindustries:32005-201
- C28, C63, C95: value 100n -> 1u; device resistor:C0603 -> rcl:C0603
- moved C28 80.3 mm to (85.0, 65.0), flipped to the bottom, turned to 0 degrees
- moved J2 26.2 mm to (2.25, 88.0), turned to 90 degrees
- moved C65 21.9 mm to (6.50, 88.0), turned to 180 degrees
- moved J1 12.4 mm to (2.25, 83.5), turned to 90 degrees
- moved C107 7.16 mm to (6.50, 83.5), turned to 0 degrees
- moved C62 5.74 mm to (90.7, 68.7)
- moved C61 5.60 mm to (85.2, 68.3)
- moved C95 5.52 mm to (63.5, 61.0), flipped to the bottom, turned to 270 degrees
- moved R64 4.28 mm to (49.1, 15.2)
- moved C156 2.00 mm to (35.9, 5.30), turned to 45 degrees
- moved C147 1.72 mm to (61.0, 6.90), turned to 180 degrees
- moved R62 1.61 mm to (56.8, 4.70), turned to 270 degrees
- moved C63 1.50 mm to (85.0, 70.0), flipped to the bottom, turned to 0 degrees
- moved C29 1.35 mm to (5.02, 73.3)
- moved R66 1.33 mm to (59.8, 4.70), turned to 270 degrees
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Connections:
- removed net ADC_SCLK: IC12.8, IC4.8, IC8.8
- removed net CONVSTART: IC12.6, IC4.6, IC8.6
- removed net PORT1TEMP: IC1.1, R14.2
- removed net PORT2TEMP: IC5.1, R26.2
- removed net REFTEMP: IC9.1, R42.2
- new net +12V: C173.1, C177.1, C185.1, IC32.12, IC32.13, IC32.30, IC32.31, J3.1
- new net FILT_IN_C1: R100.2, U2.P21
- new net FILT_IN_C2: R99.2, U2.P14
- new net FILT_OUT_C1: R104.2, U2.P16
- new net FILT_OUT_C2: R103.2, U2.P15
- new net FLACH_MOSI: U2.P64, U4.5
- new net FLASH_CLK: U2.P70, U4.6
- new net FLASH_CS: U2.P38, U4.1
- new net FLASH_MISO: R91.1, U4.2
- new net MCU_AUX1: IC33.2, U2.P55
- new net MCU_AUX2: IC33.3, U2.P51
- new net MCU_AUX3: IC33.6, U2.P50
- new net MCU_AUX4: IC33.7, U2.P48
- new net MCU_INTR: IC33.30, U2.P57
- new net MCU_MISO: IC33.27, U2.P61
- new net MCU_MOSI: IC33.28, U2.P59
- new net MCU_NSS: IC33.29, U2.P58
- new net MCU_SCK: IC33.26, U2.P56
- new net N$100: C113.2, IC28.2, IC28.3, L47.1
- new net N$161: C159.2, IC29.2, IC29.3, L48.1
- new net N$162: C168.2, IC32.1
- new net N$163: C106.2, C158.2, C160.2, C162.2, C174.1, C181.1, IC28.4, IC28.6, IC29.4, IC29.6, IC30.4, IC30.6, IC31.4, IC31.6, L51.P$2
- new net N$164: C161.2, IC30.2, IC30.3, L49.1
- new net N$165: JTAG.3, U2.P106
- new net N$166: C163.2, IC31.2, IC31.3, L50.1
- new net N$167: IC32.32, R77.2
- new net N$168: C178.2, IC32.25
- new net N$169: C178.1, IC32.28, IC32.29, L52.P$1
- new net N$170: C175.2, IC32.9
- new net N$171: C175.1, IC32.11, L53.P$1
- new net N$172: C176.2, IC32.7, R82.2
- new net N$173: JTAG.5, U2.P107
- new net N$174: C182.2, IC32.23, R79.2
- new net N$175: JTAG.9, U2.P110
- new net N$176: C183.2, IC32.22, R80.2, R81.1
- new net N$177: C170.1, C171.1, C183.1, L51.P$1, L52.P$2, R81.2
- new net N$178: C179.2, IC32.6, R83.2, R84.1
- new net N$179: C169.1, C172.1, C179.1, L53.P$2, L55.P$1, R84.2
- new net N$180: C186.2, IC32.16
- new net N$181: C186.1, IC32.14, L54.P$1
- new net N$182: C187.2, IC32.18, R85.2
- new net N$183: JTAG.1, U2.P109
- new net N$184: C188.2, IC32.19, R86.2, R87.1
- new net N$185: R88.1, X3.2
- new net N$186: R76.2, R89.2, X3.3
- new net N$187: IC33.21, R88.2
- new net N$188: IC33.22, R76.1
- new net N$189: IC33.25, R89.1
- new net N$190: IC33.24, JP1.2
- new net N$191: IC33.23, JP1.4
- new net N$192: IC33.4, JP1.5
- new net N$193: IC33.8, JP1.6
- new net N$194: R92.1, U2.P71
- new net N$195: R93.1, U2.P39
- new net N$196: R94.1, U2.P37
- new net N$197: R91.2, U2.P65
- new net N$198: R96.2, U2.P17
- new net N$199: IC16.2, R97.1, R99.1
- new net N$200: IC16.1, R100.1, R98.1
- new net N$201: IC18.1, R101.1, R103.1
- new net N$202: IC18.2, R102.1, R104.1
- new net N$203: C194.1, IC34.5, IC4.2
- new net N$204: C63.1, IC35.5, IC8.2
- new net N$205: C195.1, IC12.2, IC36.5
- new net PORT1_CONVSTART: IC4.6, U2.P134
- new net PORT1_SCLK: IC4.8, U2.P132
- new net PORT2_CONVSTART: IC8.6, U2.P47
- new net PORT2_SCLK: IC8.8, U2.P45
- new net REF_CONVSTART: IC12.6, U2.P43
- new net REF_SCLK: IC12.8, U2.P40
- new net SWITCHING_SYNC: IC32.20, R78.2, U2.P62
- new net VCCINT: C180.1, C184.1, C188.1, C208.1, C209.1, C210.1, C211.1, L54.P$2, R87.2, U2.P128, U2.P19, U2.P28, U2.P52, U2.P89
- net +3V3: now also C189.1, C190.1, C191.1, C192.1, C203.1, C204.1, C205.1, C206.1, C207.1, IC33.1, IC33.17, IC33.5, JP1.1, JTAG.4, L55.P$2, R90.2, R92.2, R93.2, R94.2, R95.2, U2.P103, U2.P122, U2.P125, U2.P129, U2.P135, U2.P18, U2.P20, U2.P31, U2.P36, U2.P4, U2.P42, U2.P53, U2.P63, U2.P69, U2.P76, U2.P86, U2.P90, U4.3, U4.7, U4.8
- net +5V/1: now also C164.2, C193.1, IC34.1, IC34.3, L47.2; no longer C28.2, IC4.2, R14.1
- net +5V/2: now also C165.2, C28.1, IC35.1, IC35.3, L48.2; no longer C63.2, IC8.2, R26.1
- net +5V/3: now also C166.2, C95.1, IC36.1, IC36.3, L49.2; no longer C95.2, IC12.2, R42.1
- net +5V/4: now also C167.2, L50.2
- net AMP_PWDN: now also U2.P24
- net ATT_D0: now also U2.P26
- net ATT_D1: now also U2.P27
- net ATT_D2: now also U2.P29
- net ATT_D3: now also U2.P30
- net ATT_D4: now also U2.P32
- net ATT_D5: now also U2.P33
- net ATT_D6: now also U2.P34
- net BAND_SELECT: now also U2.P22
- net FPGA_CLK: now also R96.1
- net GND: now also C106.1, C113.1, C158.1, C159.1, C160.1, C161.1, C162.1, C163.1, C164.1, C165.1, C166.1, C167.1, C168.1, C169.2, C170.2, C171.2, C172.2, C173.2, C174.2, C176.1, C177.2, C180.2, C181.2, C182.1, C184.2, C185.2, C187.1, C189.2, C190.2, C191.2, C192.2, C193.2, C194.2, C195.2, C203.2, C204.2, C205.2, C206.2, C207.2, C208.2, C209.2, C210.2, C211.2, C28.2, C63.2, C95.2, IC28.1, IC28.7, IC29.1, IC29.7, IC30.1, IC30.7, IC31.1, IC31.7, IC32.10, IC32.15, IC32.21, IC32.26, IC32.27, IC32.33, IC33.16, IC33.31, IC33.32, IC33.33, IC34.2, IC35.2, IC36.2, J3.3, JP1.3, JTAG.10, JTAG.2, R101.2, R102.2, R77.1, R78.1, R79.1, R80.1, R82.1, R83.1, R85.1, R86.1, R97.2, R98.2, U2.P108, U2.P113, U2.P13, U2.P130, U2.P136, U2.P25, U2.P3, U2.P49, U2.P54, U2.P60, U2.P68, U2.P73, U2.P77, U2.P91, U2.P96, U4.4, X3.5; no longer C28.1, C63.1, C95.1
- net LO1_CE: now also U2.P6
- net LO1_CLK: now also U2.P9
- net LO1_EN: now also U2.P11
- net LO1_LD: now also U2.P12
- net LO1_LE: now also U2.P7
- net LO1_MOSI: now also U2.P8
- net LO1_MUX: now also U2.P10
- net N$122: now also LP1.4; no longer LP1.1
- net N$123: now also LP1.1; no longer LP1.4
- net N$124: now also LP3.1; no longer LP3.4
- net N$125: now also LP2.1; no longer LP2.4
- net N$126: now also LP2.4; no longer LP2.1
- net N$127: now also LP3.4; no longer LP3.1
- net PORT1MIX_EN: now also U2.P137
- net PORT1_SDO: now also U2.P133
- net PORT2MIX_EN: now also U2.P44
- net PORT2_SDO: now also U2.P46
- net PORT_SELECT: now also U2.P23
- net REFMIX_EN: now also U2.P35
- net REF_SDO: now also U2.P41
- net SCL: now also IC33.19, R90.1
- net SDA: now also IC33.20, R95.1
- net SOURCE_CE: now also U2.P5
- net SOURCE_CLK: now also U2.P144
- net SOURCE_LD: now also U2.P141
- net SOURCE_LE: now also U2.P2
- net SOURCE_MOSI: now also U2.P1
- net SOURCE_MUX: now also U2.P143
- net SOURCE_RF_EN: now also U2.P142
Routing:
- net GND: track 0.00 -> 279.7 mm, vias 0 -> 135
- net +5V/1: track 0.00 -> 94.5 mm, vias 0 -> 8
- net +5V/2: track 0.00 -> 92.3 mm, vias 0 -> 8
- net +5V/3: track 0.00 -> 80.5 mm, vias 0 -> 5
- net PORT1LO1: track 0.00 -> 56.9 mm, vias 0 -> 2
- net PORT2LO2: track 0.00 -> 54.2 mm, vias 0 -> 2
- net PORT2MIX_EN: track 0.00 -> 51.0 mm, vias 0 -> 3
- net PORT1MIX_EN: track 0.00 -> 50.7 mm, vias 0 -> 3
- net REFLO1: track 0.00 -> 46.6 mm, vias 0 -> 2
- net PORT2LO1: track 0.00 -> 41.0 mm, vias 0 -> 2
- net REFMIX_EN: track 0.00 -> 39.8 mm, vias 0 -> 3
- net LO1_REF: track 0.00 -> 38.1 mm, vias 0 -> 2
- net N$160: track 0.00 -> 28.3 mm, vias 0 -> 2
- net N$154: track 0.00 -> 27.8 mm
- net +3V3: track 0.00 -> 21.6 mm
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- added copper zone on layer 2, net GND

Commit message: Routing
Parts:
- moved C125 7.24 mm to (28.0, 31.7), turned to 180 degrees
- moved R55 3.81 mm to (35.5, 27.0), turned to 90 degrees
- moved C109 1.90 mm to (21.5, 46.9)
- moved C110 1.80 mm to (36.9, 48.7), turned to 90 degrees
- moved C126 1.10 mm to (28.1, 23.4)
- moved C132 0.85 mm to (38.1, 27.6)
- moved C191 0.70 mm to (58.2, 75.5)
- moved C192 0.50 mm to (51.5, 80.5)
- moved R104 0.20 mm to (44.2, 39.1)
- moved R93 0.20 mm to (43.3, 67.5)
- turned C123 to 90 degrees
Connections:
- removed net LO1_EN: IC19.26, U2.P11
- new net LO1_RF_EN: IC19.26, U2.P143
- net ATT_D0: now also U2.P34; no longer U2.P26
- net ATT_D1: now also U2.P33; no longer U2.P27
- net ATT_D2: now also U2.P32; no longer U2.P29
- net ATT_D4: now also U2.P29; no longer U2.P32
- net ATT_D5: now also U2.P27; no longer U2.P33
- net ATT_D6: now also U2.P26; no longer U2.P34
- net FILT_IN_C1: now also U2.P16; no longer U2.P21
- net FILT_IN_C2: now also U2.P15; no longer U2.P14
- net FILT_OUT_C1: now also U2.P21; no longer U2.P16
- net FILT_OUT_C2: now also U2.P17; no longer U2.P15
- net LO1_CE: now also U2.P138; no longer U2.P6
- net LO1_CLK: now also U2.P141; no longer U2.P9
- net LO1_LD: now also U2.P142; no longer U2.P12
- net LO1_LE: now also U2.P139; no longer U2.P7
- net LO1_MOSI: now also U2.P140; no longer U2.P8
- net LO1_MUX: now also U2.P144; no longer U2.P10
- net N$198: now also U2.P14; no longer U2.P17
- net SCL: now also U2.P6
- net SDA: now also U2.P9
- net SOURCE_CE: now also U2.P1; no longer U2.P5
- net SOURCE_CLK: now also U2.P7; no longer U2.P144
- net SOURCE_LD: now also U2.P10; no longer U2.P141
- net SOURCE_MOSI: now also U2.P5; no longer U2.P1
- net SOURCE_MUX: now also U2.P8; no longer U2.P143
- net SOURCE_RF_EN: now also U2.P11; no longer U2.P142
Routing:
- net GND: track 279.7 -> 526.7 mm, vias 135 -> 202
- net +3V3: track 21.6 -> 187.9 mm, vias 0 -> 9
- net PORT_SELECT: track 0.00 -> 117.1 mm, vias 0 -> 5
- net N$163: track 12.1 -> 127.3 mm, vias 0 -> 10
- net LO1_LD: track 3.37 -> 113.0 mm, vias 1 -> 2
- net LO1_RF_EN: track 0.00 -> 109.3 mm, vias 0 -> 2
- net LO1_CLK: track 5.60 -> 106.2 mm, vias 1 -> 2
- net LO1_MUX: track 1.12 -> 100.1 mm, vias 1 -> 2
- net LO1_MOSI: track 6.76 -> 105.2 mm, vias 1 -> 2
- net LO1_LE: track 7.69 -> 105.6 mm, vias 1 -> 2
- net LO1_CE: track 9.30 -> 104.0 mm, vias 1 -> 2
- net N$156: track 0.00 -> 91.9 mm, vias 0 -> 6
- net SOURCE_CE: track 0.00 -> 64.8 mm, vias 0 -> 2
- net +5V/4: track 14.6 -> 74.1 mm, vias 0 -> 4
- net SOURCE_LE: track 0.00 -> 58.2 mm, vias 0 -> 2
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
Commit message: Routing
Parts:
- removed X3: MINI-USB-32005-201, con-cypressindustries:32005-201
- added X4: MINI-USB-SCHIELD-32005-301, con-cypressindustries:32005-301
- moved R83 3.37 mm to (73.5, 97.0), turned to 180 degrees
- moved R91 0.30 mm to (51.0, 85.0)
- moved C205 0.22 mm to (42.8, 74.4), turned to 90 degrees
- moved R92 0.22 mm to (43.8, 90.1), turned to 180 degrees
Connections:
- net GND: now also X4.5, X4.M1, X4.M2, X4.M3, X4.M4; no longer X3.5
- net N$185: now also X4.2; no longer X3.2
- net N$186: now also X4.3; no longer X3.3
Routing:
- net +3V3: track 187.9 -> 467.1 mm, vias 9 -> 34
- net GND: track 526.7 -> 804.8 mm, vias 202 -> 872
- net VCCINT: track 0.00 -> 112.2 mm, vias 0 -> 10
- net +12V: track 0.00 -> 57.7 mm, vias 0 -> 8
- net PORT2MIX_EN: track 51.0 -> 107.4 mm, vias 3 -> 4
- net N$163: track 127.3 -> 180.4 mm, vias 10 -> 16
- net PORT2_CONVSTART: track 0.00 -> 50.1 mm, vias 0 -> 2
- net PORT2_SDO: track 0.00 -> 48.9 mm, vias 0 -> 2
- net PORT2_SCLK: track 0.00 -> 48.1 mm, vias 0 -> 2
- net SCL: track 29.5 -> 76.8 mm, vias 2 -> 4
- net FLASH_CS: track 0.00 -> 41.5 mm
- net SDA: track 28.3 -> 69.5 mm, vias 2 -> 4
- net N$185: track 0.00 -> 33.8 mm, vias 0 -> 2
- net N$186: track 0.00 -> 33.7 mm, vias 0 -> 2
- net SWITCHING_SYNC: track 0.00 -> 33.1 mm, vias 0 -> 2
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- added copper zone on layer 1, net +12V
- added copper zone on layer 15, net +12V
- added copper zone on layer 15, net +3V3
- added copper zone on layer 1, net GND
- added copper zone on layer 15, net GND
- added copper zone on layer 16, net GND
- added copper zone on layer 15, net N$163
- added copper zone on layer 1, net N$169
- added copper zone on layer 1, net N$171
- added copper zone on layer 1, net N$181
- added copper zone on layer 15, net VCCINT

Commit message: Shield outline and small layout fixes
Parts:
- added LED1, LED2, LED3, LED4, LED5, LED6, LED7, LED8, LED9: (no value), led:CHIPLED_0603
- added R105, R106, R107, R108, R109, R110, R14, R26, R42: 330, VNA:R0603
- C1, C10, C104, C105, C106, C107, C108, C109, C11, C110, C113, C114, C115, C116, C117, C118, C119, C12, C120, C121, C122, C123, C124, C127, C128, C129, C13, C130, C131, C132, C133, C134, C135, C136, C137, C138, C139, C14, C140, C143, C144, C145, C146, C147, C148, C149, C150, C151, C152, C153, C154, C155, C156, C157, C158, C159, C160, C161, C162, C163, C164, C165, C166, C167, C168, C175, C176, C178, C179, C182, C183, C186, C187, C188, C191, C192, C193, C194, C195, C2, C203, C204, C205, C206, C207, C208, C209, C210, C211, C28, C3, C31, C32, C33, C34, C35, C36, C37, C38, C39, C4, C40, C41, C42, C43, C44, C5, C55, C56, C57, C58, C6, C63, C65, C66, C67, C68, C69, C7, C70, C71, C72, C73, C74, C75, C76, C8, C87, C88, C89, C9, C90, C95: device rcl:C0603 -> VNA:C0603
- C100, C101, C102, C103, C111, C112, C15, C16, C17, C18, C19, C20, C21, C22, C23, C24, C25, C26, C27, C29, C30, C45, C46, C47, C48, C49, C50, C51, C52, C53, C54, C59, C60, C61, C62, C64, C77, C78, C79, C80, C81, C82, C83, C84, C85, C86, C91, C92, C93, C94, C96, C97, C98, C99: device resistor:C0603 -> VNA:C0603
- C125, C126, C141, C142, C169, C170, C171, C172, C173, C174, C177, C180, C181, C184, C185, C189, C190: device rcl:C1206 -> VNA:C1206
- IC1, IC5, IC9: device rf:QFN65P400X400X75-17T215N -> VNA:QFN65P400X400X75-17T215N
- IC10, IC11, IC2, IC3, IC6, IC7: device rf:SON50P300X300X80-9T165X238 -> VNA:SON50P300X300X80-9T165X238
- IC12, IC4, IC8: device custom-ic:SOP50P490X110-10N -> VNA:SOP50P490X110-10N
- IC13: device rf:QFN50P400X400X90-21T270N -> VNA:QFN50P400X400X90-21T270N
- IC14, IC19: device rf:QFN50P500X500X80-33T310 -> VNA:QFN50P500X500X80-33T310
- IC15, IC20, IC34, IC35, IC36: device rf:SOT95P240X110-5 -> VNA:SOT95P240X110-5
- IC16, IC18: device rf:QFN40P180X180X55-13T76N -> VNA:QFN40P180X180X55-13T76N
- IC17, IC21: device rf:SOT230P700X180-4 -> VNA:SOT230P700X180-4
- IC22, IC25, IC26, IC27: device rf:QFN50P400X400X75-21T206 -> VNA:QFN50P400X400X75-21T206
- IC23: device rf:QFN50P400X400X75-25T270 -> VNA:QFN50P400X400X75-25T270
- IC24: device rf:SON50P200X200X80-9T90X160N -> VNA:SON50P200X200X80-9T90X160N
- IC28, IC29, IC30, IC31: device custom-ic:SON95P300X300X100-7T170X240N -> VNA:SON95P300X300X100-7T170X240N
- IC32, IC33: device custom-ic:QFN50P500X500X100-33T345N -> VNA:QFN50P500X500X100-33T345N
- J1, J2: device connector:U.FL_SMT -> VNA:U.FL_SMT
- J3: device con-jack:DCJ0202 -> VNA:DCJ0202
- JP1: device pinhead:1X06 -> VNA:1X06
- JTAG: device con-ml:ML10 -> VNA:ML10
- L1, L10, L11, L12, L13, L14, L15, L16, L17, L18, L19, L2, L20, L21, L22, L23, L24, L25, L26, L27, L28, L29, L3, L30, L31, L32, L33, L34, L35, L36, L37, L38, L39, L4, L40, L41, L42, L43, L44, L45, L46, L47, L48, L49, L5, L50, L6, L7, L8, L9: device rf:R0603 -> VNA:R0603
- L51, L52, L53, L54, L55: device custom-ic:SRN5040 -> VNA:SRN5040
- LP1, LP2, LP3: device rf:FILTRDFN160X84X70-4N -> VNA:FILTRDFN160X84X70-4N
- Q1: device crystal:FA-128 -> VNA:FA-128
- R1, R10, R11, R12, R13, R15, R16, R17, R18, R19, R2, R20, R21, R22, R23, R24, R25, R27, R28, R29, R3, R30, R31, R32, R33, R34, R35, R36, R37, R38, R39, R4, R40, R41, R43, R44, R45, R46, R47, R48, R49, R5, R6, R7, R73, R74, R75, R77, R78, R79, R8, R80, R81, R82, R83, R84, R85, R86, R87, R9: device rcl:R0603 -> VNA:R0603
- R100, R101, R102, R103, R104, R50, R51, R52, R53, R54, R55, R56, R57, R58, R59, R60, R61, R62, R63, R64, R65, R66, R67, R68, R69, R70, R71, R72, R76, R88, R89, R90, R91, R92, R93, R94, R95, R96, R97, R98, R99: device resistor:R0603 -> VNA:R0603
- T1, T2, T3: device rf:MACOM_BALUN -> VNA:MACOM_BALUN
- U2: device xilinx_devices_V6:TQ144 -> VNA:TQ144
- U4: device memory-winbond:SO08 -> VNA:SO08
- X1, X2: device rf:J502-ND-142-0711-821/826 -> VNA:J502-ND-142-0711-821/826
- X4: device con-cypressindustries:32005-301 -> VNA:32005-301
- moved C107 1.00 mm to (7.50, 83.5), flipped to the bottom, turned to 180 degrees
- moved C65 1.00 mm to (7.50, 88.0), flipped to the bottom, turned to 0 degrees
Connections:
- new net N$206: LED9.C, R14.1
- new net N$207: LED8.C, R26.1
- new net N$208: LED7.C, R42.1
- new net N$209: LED6.C, R105.1
- new net N$210: LED5.C, R106.1
- new net N$211: LED4.C, R107.1
- new net N$212: LED3.C, R108.1
- new net N$213: LED2.C, R109.1
- new net N$214: LED1.C, R110.1
- new net N$215: R14.2, U2.P105
- new net N$216: R26.2, U2.P104
- new net N$217: R42.2, U2.P99
- new net N$218: R105.2, U2.P94
- new net N$219: R106.2, U2.P85
- new net N$220: R107.2, U2.P82
- new net N$221: R108.2, U2.P75
- new net N$222: R109.2, U2.P118
- net +3V3: now also LED1.A, LED2.A, LED3.A, LED4.A, LED5.A, LED6.A, LED7.A, LED8.A, LED9.A
- net GND: now also R110.2
Routing:
- net +3V3: track 467.1 -> 503.4 mm, vias 34 -> 33
- net N$163: track 180.4 -> 144.7 mm
- net N$221: track 0.00 -> 6.32 mm
- net N$222: track 0.00 -> 5.65 mm
- net N$220: track 0.00 -> 4.69 mm
- net N$218: track 0.00 -> 4.63 mm
- net N$217: track 0.00 -> 4.07 mm
- net N$216: track 0.00 -> 3.77 mm
- net N$219: track 0.00 -> 3.57 mm
- net N$215: track 0.00 -> 3.36 mm
- net N$211: track 0.00 -> 2.22 mm
- net N$210: track 0.00 -> 2.22 mm
- net N$209: track 0.00 -> 2.22 mm
- net N$208: track 0.00 -> 2.22 mm
- net N$207: track 0.00 -> 2.22 mm
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
Commit message: Mixers disabled by default, GND plane cutouts under high-speed component pads
Parts:
- added R111, R112, R113: 10k, VNA:R0603
Connections:
- net GND: now also R111.1, R112.1, R113.1
- net PORT1MIX_EN: now also R112.2
- net PORT2MIX_EN: now also R111.2
- net REFMIX_EN: now also R113.2
Routing:
- net GND: track 806.9 -> 814.6 mm
- net REFMIX_EN: track 68.5 -> 75.6 mm
- net PORT2MIX_EN: track 107.4 -> 110.4 mm
- net PORT1MIX_EN: track 74.0 -> 75.8 mm
- added copper zone on layer 2, net N$223
- added copper zone on layer 2, net N$224
