File: Hardware/VNA.brd (EAGLE design)
At the start: 100 x 100 mm, 434 parts, among them IC1 LTC5510, IC10 LT5560, IC11 LTC6362, IC12 MCP33131D-10-E/MS, IC13 SI5351C, IC14 MAX2871, IC15 NCP702-3.3, IC16 RFSW6042, IC17 AP2114H, IC18 RFSW6042, IC19 MAX2871, IC2 LT5560, IC20 NCP702-3.3, IC21 AP2114H, IC22 F2912, IC23 F1958, IC24 TRF37A73, IC25 F2912, IC26 F2912, IC27 F2912, IC28 LDL212PU50R, IC29 LDL212PU50R, IC3 LTC6362, IC30 LDL212PU50R, IC31 LDL212PU50R, IC32 TPS65265, IC33 STM32L432KC, IC34 NCP702-1.8, IC35 NCP702-1.8, IC36 NCP702-1.8, IC4 MCP33131D-10-E/MS, IC5 LTC5510, IC6 LT5560, IC7 LTC6362, IC8 MCP33131D-10-E/MS, IC9 LTC5510, J1 U.FL-R-SMT, J2 U.FL-R-SMT, J3 DCJ0202, Q1 FA-128 26MHz, T1 MABA011082, T2 MABA011082, T3 MABA011082, U2 6SLX9TQG144, U4 W25Q16BVSN, X1 RLB DUT/RF IN, X2 RLB DUT/RF IN, X4 MINI-USB-SCHIELD-32005-301

Commit message: Testpoints + Gerber
Parts:
- added TP1, TP10, TP11, TP12, TP13, TP14, TP15, TP16, TP17, TP18, TP19, TP2, TP3, TP4, TP5, TP6, TP7, TP8, TP9: TPB1,27, testpad:B1,27
Connections:
- net +3V3: now also TP3.TP
- net +5V/1: now also TP7.TP
- net +5V/2: now also TP9.TP
- net +5V/3: now also TP11.TP
- net +5V/4: now also TP13.TP
- net GND: now also TP10.TP, TP12.TP, TP14.TP, TP6.TP, TP8.TP
- net N$110: now also TP16.TP
- net N$111: now also TP18.TP
- net N$138: now also TP19.TP
- net N$163: now also TP5.TP
- net N$203: now also TP2.TP
- net N$204: now also TP4.TP
- net N$205: now also TP15.TP
- net SOURCE_VCC: now also TP17.TP
- net VCCINT: now also TP1.TP
Routing:
- net GND: track 814.6 -> 831.6 mm
- net N$163: track 144.7 -> 154.3 mm, vias 16 -> 17
- net +3V3: track 503.4 -> 509.9 mm
- net +5V/4: track 74.1 -> 77.6 mm
- net VCCINT: track 112.2 -> 115.2 mm
- net N$205: track 4.32 -> 7.36 mm
- net N$203: track 4.44 -> 7.44 mm
- net N$204: track 4.28 -> 7.23 mm
- net SOURCE_VCC: track 37.4 -> 40.1 mm
- net +5V/2: track 92.3 -> 95.1 mm
- net +5V/1: track 94.6 -> 97.2 mm
- net N$138: track 16.3 -> 18.6 mm
- net N$110: track 14.3 -> 16.7 mm
- net N$111: track 9.86 -> 11.7 mm
- net +5V/3: track 84.0 -> 85.9 mm
Other:
- board text added: "GND"

Commit message: BOM + AUX4->RESET
Connections:
- net MCU_AUX4 renamed FPGA_RESET
Changed lines of the file:
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@@
 <drawing>
 <settings>
-<setting alwaysvectorfont="yes"/>
+<setting alwaysvectorfont="no"/>
 <setting verticaltext="up"/>
 </settings>
@@
 <wire x1="51.25" y1="76.75" x2="51.75" y2="77.25" width="0.3" layer="1"/>
 </signal>
-<signal name="MCU_AUX4">
+<signal name="FPGA_RESET">
 <contactref element="IC33" pad="7"/>
 <contactref element="U2" pad="P48"/>

Commit message: Bugfixes
Connections:
- net FILT_IN_C1: now also R99.2, U2.P15; no longer R100.2, U2.P16
- net FILT_IN_C2: now also R100.2, U2.P16; no longer R99.2, U2.P15
Routing:
- net FILT_IN_C2: track 40.2 -> 48.5 mm
- net FILT_IN_C1: track 48.5 -> 40.2 mm
Changed lines of the file:
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@@
 <wire x1="43.1" y1="33" x2="42.9" y2="32.8" width="0.3" layer="16"/>
 </signal>
-<signal name="FILT_IN_C1">
+<signal name="FILT_IN_C2">
 <contactref element="R100" pad="2"/>
 <wire x1="46.35" y1="31.5" x2="47.5" y2="31.5" width="0.3" layer="16"/>
@@
 <wire x1="40.4" y1="39.1" x2="45.3" y2="39.1" width="0.3" layer="16"/>
 </signal>
-<signal name="FILT_IN_C2">
+<signal name="FILT_IN_C1">
 <contactref element="R99" pad="2"/>
 <wire x1="38.65" y1="31.5" x2="38.1" y2="31.5" width="0.3" layer="16"/>

Commit message: Part values of final IF filter adjusted
Parts:
- C16, C17, C19, C60, C61, C62, C92, C93, C94: value 22n -> 330p
- C27, C53, C85: value 4n7 -> 330p
- L19, L20, L29, L30, L4, L5: value 4u7 -> 220Ohm
- R17, R18, R29, R30: value 620 -> 6k8
- R19, R20, R31, R32, R47, R48: value 33 -> 220
- R45, R46: value 200 -> 4k7

Commit message: Lowband source implemented, faster algorithm for PLL divider selection
Parts:
- R73, R75: value TBD -> 100
- R74: value TBD -> 62
Changed lines of the file:
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@@
 <attribute name="VALUE" x="18.89" y="1.27" size="1.778" layer="27" rot="R90"/>
 </element>
-<element name="R73" library="VNA" library_urn="urn:adsk.eagle:library:19762030" package="R0603" package3d_urn="urn:adsk.eagle:package:19762122/2" value="TBD" x="36.5" y="48" smashed="yes">
+<element name="R73" library="VNA" library_urn="urn:adsk.eagle:library:19762030" package="R0603" package3d_urn="urn:adsk.eagle:package:19762122/2" value="100" x="36.5" y="48" smashed="yes">
 <attribute name="VALUE" x="35.865" y="46.095" size="1.27" layer="27"/>
 </element>
-<element name="R74" library="VNA" library_urn="urn:adsk.eagle:library:19762030" package="R0603" package3d_urn="urn:adsk.eagle:package:19762122/2" value="TBD" x="35.5" y="50.5" smashed="yes" rot="R90">
+<element name="R74" library="VNA" library_urn="urn:adsk.eagle:library:19762030" package="R0603" package3d_urn="urn:adsk.eagle:package:19762122/2" value="62" x="35.5" y="50.5" smashed="yes" rot="R90">
 <attribute name="VALUE" x="37.405" y="49.865" size="1.27" layer="27" rot="R90"/>
 </element>
-<element name="R75" library="VNA" library_urn="urn:adsk.eagle:library:19762030" package="R0603" package3d_urn="urn:adsk.eagle:package:19762122/2" value="TBD" x="37.5" y="50.5" smashed="yes" rot="R90">
+<element name="R75" library="VNA" library_urn="urn:adsk.eagle:library:19762030" package="R0603" package3d_urn="urn:adsk.eagle:package:19762122/2" value="100" x="37.5" y="50.5" smashed="yes" rot="R90">
 <attribute name="VALUE" x="39.405" y="49.865" size="1.27" layer="27" rot="R90"/>
 </element>
